File: scriptPad_PCB/scriptPad_PCB.kicad_pcb (KiCad board)
At the start: 2 copper layers, 287.3 x 111.3 mm, 83 parts, among them SW2 TS365CA, SW3 EC11E0940501, SW4 TS365CA, U1 RP2040, U16 74HCT1G125GV,125, U2 AP2112K-3.3, U3 W25Q32JVZP, X1 X322512MSB4SI

Commit message: Updating PCB to new version
Parts:
- removed the ? at (307.7, 147.1)
- removed the ? at (307.7, 44.2)
- removed the G*** at (167.9, 95.4)
- removed the G*** at (264.5, 94.1)
- removed the SW3 at (106.9, 61.0)
- added ?: , , F.Cu at (234.8, 44.1)
- added ?: , , F.Cu at (234.8, 147.1)
- added G***: LOGO, Graphics:frontGraphics, F.Cu at (167.4, 95.5)
- added J1: Conn_01x05_Pin, Connector_PinHeader_1.27mm:PinHeader_1x05_P1.27mm_Vertical, B.Cu at (116.8, 85.1)
- added R1: 5.1K, Resistor_SMD:R_0603_1608Metric, B.Cu at (70.4, 50.8)
- added R11: 22, Resistor_SMD:R_0603_1608Metric, B.Cu at (71.9, 50.8)
- added R12: 22, Resistor_SMD:R_0603_1608Metric, B.Cu at (73.4, 50.8)
- added R2: 5.1K, Resistor_SMD:R_0603_1608Metric, B.Cu at (75.0, 50.8)
- added SW1: ED11301M-FB12A4.0-C20-102-G219, easyeda2kicad:SW-TH_CTR_ED11301M-FB12A4.0-C20-102-G219, F.Cu at (106.9, 61.0)
- added TP1: TP_USB-, TestPoint:TestPoint_Pad_D2.0mm, F.Cu at (66.5, 51.8)
- added TP10: TP_SW, TestPoint:TestPoint_Pad_D2.0mm, F.Cu at (105.4, 48.3)
- added TP11: TP_ROTA, TestPoint:TestPoint_Pad_D2.0mm, F.Cu at (104.4, 74.9)
- added TP12: TP_ROTB, TestPoint:TestPoint_Pad_D2.0mm, F.Cu at (109.2, 74.9)
- added TP13: TestPoint, TestPoint:TestPoint_Pad_D2.0mm, F.Cu at (69.1, 71.1)
- added TP14: TestPoint, TestPoint:TestPoint_Pad_D2.0mm, F.Cu at (69.1, 68.1)
- added TP15: TestPoint, TestPoint:TestPoint_Pad_D2.0mm, F.Cu at (69.1, 65.0)
- added TP16: TestPoint, TestPoint:TestPoint_Pad_D2.0mm, F.Cu at (69.1, 62.0)
- added TP17: TestPoint, TestPoint:TestPoint_Pad_D2.0mm, F.Cu at (69.1, 58.9)
- added TP18: TestPoint, TestPoint:TestPoint_Pad_D2.0mm, F.Cu at (41.7, 88.9)
- added TP19: TestPoint, TestPoint:TestPoint_Pad_D2.0mm, F.Cu at (62.5, 88.9)
- added TP2: TP_USB+, TestPoint:TestPoint_Pad_D2.0mm, F.Cu at (79.2, 51.8)
- added TP20: TestPoint, TestPoint:TestPoint_Pad_D2.0mm, F.Cu at (82.8, 88.9)
- added TP21: TestPoint, TestPoint:TestPoint_Pad_D2.0mm, F.Cu at (103.1, 88.9)
- added TP22: TestPoint, TestPoint:TestPoint_Pad_D2.0mm, F.Cu at (31.0, 88.9)
- added TP23: TestPoint, TestPoint:TestPoint_Pad_D2.0mm, F.Cu at (31.0, 112.3)
- added TP24: TestPoint, TestPoint:TestPoint_Pad_D2.0mm, F.Cu at (31.0, 132.1)
- added TP3: TP_5V, TestPoint:TestPoint_Pad_D2.0mm, F.Cu at (81.8, 43.7)
- added TP4: TP_3.3V, TestPoint:TestPoint_Pad_D2.0mm, F.Cu at (91.4, 43.7)
- added TP5: TP_GND, TestPoint:TestPoint_Pad_D2.0mm, F.Cu at (98.3, 43.7)
- added TP6: TP_CS, TestPoint:TestPoint_Pad_D2.0mm, F.Cu at (58.4, 47.0)
- added TP7: TP_MOSI, TestPoint:TestPoint_Pad_D2.0mm, F.Cu at (54.6, 47.0)
- added TP8: TP_CLK, TestPoint:TestPoint_Pad_D2.0mm, F.Cu at (50.8, 47.0)
- added TP9: TP_MISO, TestPoint:TestPoint_Pad_D2.0mm, F.Cu at (47.0, 47.0)
- U3: footprint Package_SON:WSON-8-1EP_6x5mm_P1.27mm_EP3.4x4.3mm -> easyeda2kicad:SOIC-8_L5.3-W5.3-P1.27-LS8.0-BL
- moved U3 3.75 mm to (103.4, 48.5), turned to -90 degrees
- moved R3 2.44 mm to (110.6, 47.5), turned to 90 degrees
- moved C9 1.09 mm to (103.1, 63.1)
- moved ? 0.63 mm to (211.3, 44.2)
- moved H4 0.63 mm to (211.3, 147.1)
- moved ? 0.28 mm to (124.8, 43.9)
- moved H1 0.18 mm to (115.6, 44.1)
- moved ? 0.13 mm to (220.5, 44.1)
- moved ? 0.13 mm to (220.5, 147.1)
- moved H4 0.13 mm to (115.6, 147.1)
- moved H2 0.13 mm to (28.4, 44.1)
- moved H3 0.13 mm to (28.4, 147.1)
- renumbered SW4 to SW3, U16 to U4
Connections:
- U1 pad 2: unconnected-(U1-GPIO0-Pad2) -> RX
- U1 pad 24: unconnected-(U1-SWCLK-Pad24) -> SWCLK
- U1 pad 25: unconnected-(U1-SWD-Pad25) -> SWD
- U1 pad 3: unconnected-(U1-GPIO1-Pad3) -> TX
- USBC1 pad A5: unconnected-(USBC1-CC1-PadA5) -> Net-(USBC1-CC1)
- USBC1 pad A6: USB_D+ -> /DP
- USBC1 pad A7: USB_D- -> /DN
- USBC1 pad B5: unconnected-(USBC1-CC2-PadB5) -> Net-(USBC1-CC2)
- USBC1 pad B6: USB_D+ -> /DP
- USBC1 pad B7: USB_D- -> /DN
Routing:
- net GND: track 68.8 -> 167.6 mm, vias 12 -> 13
- net RX: track 0.00 -> 49.0 mm, vias 0 -> 3
- net TX: track 0.00 -> 47.3 mm, vias 0 -> 1
- net SWD: track 0.00 -> 45.9 mm, vias 0 -> 1
- net SWCLK: track 0.00 -> 38.4 mm, vias 0 -> 1
- net LCD_RESET: track 21.0 -> 42.1 mm, vias 2 -> 3
- net SD_MOSI: track 62.0 -> 77.7 mm, vias 4 -> 5
- net LCD_DC: track 22.3 -> 36.2 mm, vias 2 -> 3
- net KB_COL1: track 90.8 -> 103.6 mm, vias 0 -> 1
- net SD_CS: track 56.9 -> 68.5 mm, vias 2 -> 4
- net LCD_DIN: track 30.4 -> 42.0 mm, vias 2 -> 3
- net +3.3V: track 233.7 -> 244.6 mm, vias 10 -> 12
- net KB_COL2: track 87.5 -> 97.4 mm, vias 0 -> 1
- net KB_COL3: track 108.3 -> 117.7 mm, vias 0 -> 1
- net LCD_CS: track 29.5 -> 38.8 mm, vias 2 -> 3
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Other:
- board size 287.3 x 111.3 mm -> 219.7 x 111.3 mm
- board text added: "DEBUG ME!"
- board text added: "GND"
- board text added: "R5"
- board text added: "RX"
- board text added: "SWCLK"
- board text added: "SWD"
- board text added: "TX"
