File: scriptPad_PCB/scriptPad_PCB.kicad_sch (KiCad schematic)
At the start: 73 parts, among them SW2 TS365CA, SW3 EC11E0940501, SW4 TS365CA, U1 RP2040, U16 74HCT1G125GV,125, U2 AP2112K-3.3, U3 W25Q32JVZP, X1 X322512MSB4SI

Commit message: Updating PCB to new version
Parts:
- removed SW3: EC11E0940501, easyeda2kicad:SW-SMD_EC11E0940501, symbol easyeda2kicad:EC11E0940501
- added J1: Conn_01x05_Pin, Connector_PinHeader_1.27mm:PinHeader_1x05_P1.27mm_Vertical, symbol Connector:Conn_01x05_Pin
- added R1, R2: 5.1K, Resistor_SMD:R_0603_1608Metric, symbol Device:R
- added R11, R12: 22, Resistor_SMD:R_0603_1608Metric, symbol Device:R
- added SW1: ED11301M-FB12A4.0-C20-102-G219, easyeda2kicad:SW-TH_CTR_ED11301M-FB12A4.0-C20-102-G219, symbol easyeda2kicad:ED11301M-FB12A4.0-C20-102-G219
- added TP1: TP_USB-, TestPoint:TestPoint_Pad_D2.0mm, symbol Connector:TestPoint
- added TP10: TP_SW, TestPoint:TestPoint_Pad_D2.0mm, symbol Connector:TestPoint
- added TP11: TP_ROTA, TestPoint:TestPoint_Pad_D2.0mm, symbol Connector:TestPoint
- added TP12: TP_ROTB, TestPoint:TestPoint_Pad_D2.0mm, symbol Connector:TestPoint
- added TP13, TP14, TP15, TP16, TP17, TP18, TP19, TP20, TP21, TP22, TP23, TP24: TestPoint, TestPoint:TestPoint_Pad_D2.0mm, symbol Connector:TestPoint
- added TP2: TP_USB+, TestPoint:TestPoint_Pad_D2.0mm, symbol Connector:TestPoint
- added TP3: TP_5V, TestPoint:TestPoint_Pad_D2.0mm, symbol Connector:TestPoint
- added TP4: TP_3.3V, TestPoint:TestPoint_Pad_D2.0mm, symbol Connector:TestPoint
- added TP5: TP_GND, TestPoint:TestPoint_Pad_D2.0mm, symbol Connector:TestPoint
- added TP6: TP_CS, TestPoint:TestPoint_Pad_D2.0mm, symbol Connector:TestPoint
- added TP7: TP_MOSI, TestPoint:TestPoint_Pad_D2.0mm, symbol Connector:TestPoint
- added TP8: TP_CLK, TestPoint:TestPoint_Pad_D2.0mm, symbol Connector:TestPoint
- added TP9: TP_MISO, TestPoint:TestPoint_Pad_D2.0mm, symbol Connector:TestPoint
- C1, C2: LCSC (none) -> C17024
- C3: LCSC (none) -> C19110
- C4: LCSC (none) -> C1591
- D1: LCSC (none) -> C2891733
- SW_CN1, SW_CN10, SW_CN11, SW_CN12, SW_CN2, SW_CN3, SW_CN4, SW_CN5, SW_CN6, SW_CN7, SW_CN8, SW_CN9: footprint Switch_Keyboard_Hotswap_Kailh:SW_Hotswap_Kailh_MX_1.00u -> easyeda2kicad:SMD_KEYBOARD-SW
- U2: LCSC (none) -> C51118
- renumbered SW4 to SW3, U16 to U4
Connections:
- net +3.3V: now also TP4.1
- net +5V: now also TP3.1
- net GND: now also J1.3 (Pin_3), R1.2, R2.2, SW1.4 (SW2.2), SW1.C, SW1.S1, SW1.S2, TP5.1
- net KB_COL0: now also TP21.1
- net KB_COL1: now also TP20.1
- net KB_COL2: now also TP19.1
- net KB_COL3: now also TP18.1
- net KB_ROW0: now also TP22.1
- net KB_ROW1: now also TP23.1
- net KB_ROW2: now also TP24.1
- net LCD_CLK: now also TP16.1
- net LCD_CS: now also TP14.1
- net LCD_DC: now also TP15.1
- net LCD_DIN: now also TP13.1
- net LCD_RESET: now also TP17.1
- net ROT_1: now also SW1.A, TP11.1
- net ROT_2: now also SW1.B, TP12.1
- net ROT_SW: now also SW1.3 (SW2.1), TP10.1
- net SD_CLK: now also TP8.1
- net SD_CS: now also TP6.1
- net SD_MISO: now also TP9.1
- net SD_MOSI: now also TP7.1
- net USB_D+: now also R12.2, TP2.1; no longer USBC1.A6 (DP1), USBC1.B6 (DP2)
- net USB_D-: now also R11.2, TP1.1; no longer USBC1.A7 (DN1), USBC1.B7 (DN2)
- net RX: now reaches U1.2 (GPIO0)
- net RX: now also J1.2 (Pin_2)
- net SWCLK: now reaches U1.24 (SWCLK)
- net SWCLK: now also J1.4 (Pin_4)
- net SWD: now reaches U1.25 (SWD)
- net SWD: now also J1.5 (Pin_5)
- net TX: now reaches U1.3 (GPIO1)
- net TX: now also J1.1 (Pin_1)
- net at USBC1.A5 (CC1): now also R1.1
- net at USBC1.B5 (CC2): now also R2.1
- new net DN: R11.1, USBC1.A7 (DN1), USBC1.B7 (DN2)
- new net DP: R12.1, USBC1.A6 (DP1), USBC1.B6 (DP2)
Other:
- note added: "DEBUGGER"
- moved on the sheet: C5, C6, FPC1, R5, X1
